Commit message: Zed camera added to p3dx robot

File: src/p3dx_clone/p3dx_description/urdf/p3dx/pioneer3dx.xacro (robot description, xacro)
@@ -7,4 +7,9 @@
   <xacro:include filename="$(find p3dx_description)/urdf/p3dx/pioneer3dx_body.xacro"/>
   <xacro:pioneer3dx_body name="chassis" parent="base_link" meshes="package://p3dx_description/meshes/p3dx"/>
+  <!-- ZED Camera -->
+  <xacro:include filename="$(find zed_description)/urdf/zed_descr.urdf.xacro"/>
+  <xacro:stereolabs_camera parent="chassis">
+    <origin xyz="0 0 1.0" rpy="0 0 0"/>
+  </xacro:stereolabs_camera>
   <!-- Hokuyo UTM-30LX -->
   <xacro:include filename="$(find p3dx_description)/urdf/sensors/hokuyo_utm30lx.urdf.xacro" />
